Commit message: robot urdf/sdf with both robot arms

File: install/mechelangelo_description/share/mechelangelo_description/urdf/mechelangelo_arm.urdf (robot description, URDF)
Before this commit: robot mechelangelo_arm, 8 links, 7 joints
Joints:
- joint base_fixed_joint: origin xyz=0 0 0.05 rpy=0 0 0 -> xyz=0 0 0.05 rpy=1.5708 0 0
