Commit message: urdf done, world imported, need to start sdf

File: src/mechelangelo_description/urdf/mechelangelo_base.urdf (robot description, URDF)
Before this commit: robot mechelangelo, 3 links, 2 joints
Links:
- added link base_scan, mass 0.114; visual mesh filename=package://mechelangelo_description/meshes/sensors/lds.stl scale=0.001 0.001 0.001
- added link camera_link, mass 0.05; collision box size=0.015 0.030 0.027; visual box size=0.015 0.030 0.027
- added link camera_rgb_frame
- added link camera_rgb_optical_frame
- added link caster_link, mass 0.2; collision sphere radius=0.03; visual sphere radius=0.03
- added link imu_link, mass 0.01
- link base_link: geometry collision mesh filename=package://mechelangelo_description/meshes/base/base.stl scale=0.001 0.001 0.001; visual mesh filename=package://mechelangelo_description/meshes/base/base.stl scale=0.001 0.001 0.001
- link left_wheel_link: geometry collision cylinder length=0.03 radius=0.075; visual mesh filename=package://mechelangelo_description/meshes/wheels/wheel.stl scale=0.001 0.001 0.001
- link right_wheel_link: geometry collision cylinder length=0.03 radius=0.075; visual mesh filename=package://mechelangelo_description/meshes/wheels/wheel.stl scale=0.001 0.001 0.001
Joints:
- added joint camera_joint: type fixed, parent base_link, child camera_link, origin xyz=0 0 1.480 rpy=0 0 0
- added joint camera_rgb_joint: type fixed, parent camera_link, child camera_rgb_frame, origin xyz=0 0 0 rpy=0 0 0
- added joint camera_rgb_optical_joint: type fixed, parent camera_rgb_frame, child camera_rgb_optical_frame, origin xyz=0 0 0 rpy=-1.5708 0 -1.5708
- added joint caster_joint: type fixed, parent base_link, child caster_link, origin xyz=-0.18 0.0 0.03 rpy=0 0 0
- added joint imu_joint: type fixed, parent base_link, child imu_link, origin xyz=0.0 0 0.068 rpy=0 0 0
- added joint scan_joint: type fixed, parent base_link, child base_scan, origin xyz=0 0 0.280 rpy=0 0 0

Commit message: urdf somehwat fixed, sdf needs to be fixed helicopter issue

File: src/mechelangelo_description/urdf/mechelangelo_base.urdf (robot description, URDF)
Before this commit: robot mechelangelo, 9 links, 8 joints
Links:
- link base_link: geometry collision mesh filename=package://mechelangelo_description/meshes/base/base.dae scale=1 1 1; visual mesh filename=package://mechelangelo_description/meshes/base/base.dae scale=1 1 1
- link base_scan: geometry visual mesh filename=package://mechelangelo_description/meshes/sensors/lds.stl scale=1 1 1
- link left_wheel_link: geometry collision cylinder length=0.03 radius=0.075; visual mesh filename=package://mechelangelo_description/meshes/wheels/wheel.dae scale=1 1 1
- link right_wheel_link: geometry collision cylinder length=0.03 radius=0.075; visual mesh filename=package://mechelangelo_description/meshes/wheels/wheel.dae scale=1 1 1
Joints:
- joint left_wheel_joint: origin xyz=0.11091 0.20103 0.075 rpy=0 0 0 -> xyz=0 0 0 rpy=0 0 0
- joint right_wheel_joint: origin xyz=0.11091 -0.20103 0.075 rpy=0 0 0 -> xyz=0 0 0 rpy=0 0 0

Commit message: IMU integration first attempt, working in sim]

File: src/mechelangelo_description/urdf/mechelangelo_base.urdf (robot description, URDF)
Before this commit: robot mechelangelo, 9 links, 8 joints
Joints:
- joint imu_joint: origin xyz=0.0 0 0.068 rpy=0 0 0 -> xyz=0 0 0.37 rpy=0 0 0
