Commit message: model fixed to have joint 3 arm movement, set poses calculated in sim, need to run full run tests

File: src/mechelangelo_description/urdf/mechelangelo_final.urdf (robot description, URDF)
Before this commit: robot mechelangelo_final, 18 links, 17 joints
Links:
- link left_hand_link: geometry collision box size=0.08 0.12 0.08; visual mesh filename=package://mechelangelo_description/meshes/Arms/hand_part_DA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 scale=1 1 1
- link left_id1_link: geometry collision box size=0.075 0.09337 0.075; visual mesh filename=package://mechelangelo_description/meshes/Arms/ID1_DAE/ID1.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 scale=1 1 1
- link left_id2_link: geometry collision box size=0.09 0.40287 0.09; visual mesh filename=package://mechelangelo_description/meshes/Arms/ID2_DAE/id2.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 scale=1 1 1
- link left_id3_link: geometry collision box size=0.09 0.09337 0.09; visual mesh filename=package://mechelangelo_description/meshes/Arms/ID3_Dae/ID3.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 scale=1 1 1
- link left_id4_link: geometry collision box size=0.12 0.12 0.12; visual mesh filename=package://mechelangelo_description/meshes/Arms/ID4_Dae/ID4.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 scale=1 1 1
- link right_hand_link: geometry collision box size=0.08 0.12 0.08; visual mesh filename=package://mechelangelo_description/meshes/Arms/hand_part_DA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 scale=1 1 1
- link right_id1_link: geometry collision box size=0.075 0.09337 0.075; visual mesh filename=package://mechelangelo_description/meshes/Arms/ID1_DAE/ID1.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 scale=1 1 1
- link right_id2_link: geometry collision box size=0.09 0.40287 0.09; visual mesh filename=package://mechelangelo_description/meshes/Arms/ID2_DAE/id2.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 scale=1 1 1
- link right_id3_link: geometry collision box size=0.09 0.09337 0.09; visual mesh filename=package://mechelangelo_description/meshes/Arms/ID3_Dae/ID3.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 scale=1 1 1
- link right_id4_link: geometry collision box size=0.12 0.12 0.12; visual mesh filename=package://mechelangelo_description/meshes/Arms/ID4_Dae/ID4.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 scale=1 1 1
Joints:
- joint left_joint3: axis (none) -> 0 0 1; limit (none) -> lower=-2.0944 upper=2.0944 effort=15 velocity=1.5; type fixed -> revolute
- joint right_joint3: axis (none) -> 0 0 -1; limit (none) -> lower=-2.0944 upper=2.0944 effort=15 velocity=1.5; type fixed -> revolute
