Commit message: arms moving joint 3 fixed so angles are publishing wrong

File: scratch/packages/model files/URDFbeforejointlimits.urdf (robot description, URDF)
Before this commit: robot mechelangelo_final, 18 links, 17 joints
Links:
- link left_hand_link: geometry collision mesh filename=package://mechelangelo_description/meshes/Arms/hand part DA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 scale=1 1 1; visual mesh filename=package://mechelangelo_description/meshes/Arms/hand part DA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 scale=1 1 1
- link left_id1_link: geometry collision mesh filename=package://mechelangelo_description/meshes/Arms/ID1 DAE/ID1.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 scale=1 1 1; visual mesh filename=package://mechelangelo_description/meshes/Arms/ID1 DAE/ID1.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 scale=1 1 1
- link left_id2_link: geometry collision mesh filename=package://mechelangelo_description/meshes/Arms/ID2 DAE/id2.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 scale=1 1 1; visual mesh filename=package://mechelangelo_description/meshes/Arms/ID2 DAE/id2.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 scale=1 1 1
- link left_id3_link: geometry collision mesh filename=package://mechelangelo_description/meshes/Arms/ID3 Dae/ID3.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 scale=1 1 1; visual mesh filename=package://mechelangelo_description/meshes/Arms/ID3 Dae/ID3.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 scale=1 1 1
- link left_id4_link: geometry collision mesh filename=package://mechelangelo_description/meshes/Arms/ID4 Dae/ID4.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 scale=1 1 1; visual mesh filename=package://mechelangelo_description/meshes/Arms/ID4 Dae/ID4.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 scale=1 1 1
- link right_hand_link: geometry collision mesh filename=package://mechelangelo_description/meshes/Arms/hand part DA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 scale=1 1 1; visual mesh filename=package://mechelangelo_description/meshes/Arms/hand part DA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 scale=1 1 1
- link right_id1_link: geometry collision mesh filename=package://mechelangelo_description/meshes/Arms/ID1 DAE/ID1.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 scale=1 1 1; visual mesh filename=package://mechelangelo_description/meshes/Arms/ID1 DAE/ID1.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 scale=1 1 1
- link right_id2_link: geometry collision mesh filename=package://mechelangelo_description/meshes/Arms/ID2 DAE/id2.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 scale=1 1 1; visual mesh filename=package://mechelangelo_description/meshes/Arms/ID2 DAE/id2.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 scale=1 1 1
- link right_id3_link: geometry collision mesh filename=package://mechelangelo_description/meshes/Arms/ID3 Dae/ID3.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 scale=1 1 1; visual mesh filename=package://mechelangelo_description/meshes/Arms/ID3 Dae/ID3.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 scale=1 1 1
- link right_id4_link: geometry collision mesh filename=package://mechelangelo_description/meshes/Arms/ID4 Dae/ID4.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 scale=1 1 1; visual mesh filename=package://mechelangelo_description/meshes/Arms/ID4 Dae/ID4.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 scale=1 1 1
Joints:
- joint left_hand_joint: axis 1 0 0 -> 0 1 0; limit lower=-2.0944 upper=2.0944 effort=10 velocity=1.0 -> lower=-1.5708 upper=1.5708 effort=10 velocity=1.0
- joint left_joint1: limit lower=-2.0944 upper=2.0944 effort=25 velocity=1.5 -> lower=-3.1416 upper=3.1416 effort=25 velocity=1.5
- joint left_joint2: axis 1 0 0 -> 0 1 0; limit lower=-2.0944 upper=2.0944 effort=20 velocity=1.5 -> lower=-3.1416 upper=3.1416 effort=20 velocity=1.5
- joint right_hand_joint: axis -1 0 0 -> 0 1 0; limit lower=-2.0944 upper=2.0944 effort=10 velocity=1.0 -> lower=-1.5708 upper=1.5708 effort=10 velocity=1.0
- joint right_joint1: limit lower=-2.0944 upper=2.0944 effort=25 velocity=1.5 -> lower=-3.1416 upper=3.1416 effort=25 velocity=1.5
- joint right_joint2: axis -1 0 0 -> 0 1 0; limit lower=-2.0944 upper=2.0944 effort=20 velocity=1.5 -> lower=-3.1416 upper=3.1416 effort=20 velocity=1.5

File: scratch/packages/model files/urdfbeforecontroller.urdf (robot description, URDF)
Before this commit: robot mechelangelo_final, 18 links, 17 joints
Links:
- link left_hand_link: geometry collision mesh filename=package://mechelangelo_description/meshes/Arms/hand part DA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 scale=1 1 1; visual mesh filename=package://mechelangelo_description/meshes/Arms/hand part DA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 scale=1 1 1
- link left_id1_link: geometry collision mesh filename=package://mechelangelo_description/meshes/Arms/ID1 DAE/ID1.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 scale=1 1 1; visual mesh filename=package://mechelangelo_description/meshes/Arms/ID1 DAE/ID1.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 scale=1 1 1
- link left_id2_link: geometry collision mesh filename=package://mechelangelo_description/meshes/Arms/ID2 DAE/id2.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 scale=1 1 1; visual mesh filename=package://mechelangelo_description/meshes/Arms/ID2 DAE/id2.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 scale=1 1 1
- link left_id3_link: geometry collision mesh filename=package://mechelangelo_description/meshes/Arms/ID3 Dae/ID3.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 scale=1 1 1; visual mesh filename=package://mechelangelo_description/meshes/Arms/ID3 Dae/ID3.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 scale=1 1 1
- link left_id4_link: geometry collision mesh filename=package://mechelangelo_description/meshes/Arms/ID4 Dae/ID4.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 scale=1 1 1; visual mesh filename=package://mechelangelo_description/meshes/Arms/ID4 Dae/ID4.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 scale=1 1 1
- link right_hand_link: geometry collision mesh filename=package://mechelangelo_description/meshes/Arms/hand part DA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 scale=1 1 1; visual mesh filename=package://mechelangelo_description/meshes/Arms/hand part DA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 scale=1 1 1
- link right_id1_link: geometry collision mesh filename=package://mechelangelo_description/meshes/Arms/ID1 DAE/ID1.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 scale=1 1 1; visual mesh filename=package://mechelangelo_description/meshes/Arms/ID1 DAE/ID1.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 scale=1 1 1
- link right_id2_link: geometry collision mesh filename=package://mechelangelo_description/meshes/Arms/ID2 DAE/id2.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 scale=1 1 1; visual mesh filename=package://mechelangelo_description/meshes/Arms/ID2 DAE/id2.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 scale=1 1 1
- link right_id3_link: geometry collision mesh filename=package://mechelangelo_description/meshes/Arms/ID3 Dae/ID3.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 scale=1 1 1; visual mesh filename=package://mechelangelo_description/meshes/Arms/ID3 Dae/ID3.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 scale=1 1 1
- link right_id4_link: geometry collision mesh filename=package://mechelangelo_description/meshes/Arms/ID4 Dae/ID4.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 scale=1 1 1; visual mesh filename=package://mechelangelo_description/meshes/Arms/ID4 Dae/ID4.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 scale=1 1 1
Joints:
- joint left_hand_joint: axis 1 0 0 -> 0 1 0
- joint left_joint2: axis 1 0 0 -> 0 1 0
- joint right_hand_joint: axis -1 0 0 -> 0 1 0
- joint right_joint2: axis -1 0 0 -> 0 1 0
